Commit message: 200323

File: urdf/gripper_base.xacro (robot description, xacro)
@@ -5,4 +5,6 @@
 <robot name="gripper_base" xmlns:xacro="http://www.ros.org/wiki/xacro">>
   <xacro:include filename="$(find gripper_base)/urdf/gripper_base.gazebo"/>
+  <!-- <xacro:include filename="$(find fingertest)/urdf/fingertest.xacro"/> -->
+<xacro:macro name="gripper_base" params="parent child *origin">
   <link
     name="gripper_base_link">
@@ -85,11 +87,9 @@
     </collision>
   </link>
-  <link name="world"/>
+  <!-- <link name="world"/> -->
   <joint name="fixed123" type="fixed">
-    <origin
-      xyz="0 0 0"
-      rpy="0 0 0" />
+    <xacro:insert_block name="origin" />
     <parent
-      link="world" />
+      link="${parent}" />
     <child
       link="gripper_base_link" />
@@ -160,6 +160,8 @@
     <child
       link="r_finger_link" />
+    <!-- <axis
+      xyz="0 0 -1" /> -->
     <axis
-      xyz="0 0 -1" />
+      xyz="0 0 1" />
   </joint>
   <transmission name="tran1">
@@ -183,3 +185,5 @@
     </actuator>
   </transmission>
+<xacro:gripper_base_gazebo/>
+</xacro:macro>
 </robot>
